File: qcopter_fea_bb.sch (EAGLE design)
At the start: 11 parts, among them U1 ADAFRUIT_FEATHER_32U4_RFM

Commit message: QCOPTER rev. A
QCOPTER rev. A
Parts:
- added R3, R4, R5: 100K, resistor:R-EU_0207/10
- added R6: 1K, resistor:R-EU_0207/10
Connections:
- new net N$1: JP6.5, R6.2
- net +3V3: now also R3.2, R4.2, R5.2
- net CS_A/G: now also R3.1
- net CS_ALT: now also R5.1
- net CS_M: now also R4.1
- net ESC1_S: now also JP1.1; no longer JP1.3
- net ESC4_S: now also JP4.1; no longer JP4.3
- net GND: now also JP1.3, JP4.3; no longer JP1.1, JP4.1
- net MISO: now also R6.1; no longer JP6.5
Other:
- note added: "A"
- note added: "QCOPTER"
- note removed: "draft"
- moved on the sheet: JP2, JP3, JP4

Commit message: R1, R2 = 100K, C1 = 0,33F
R1, R2 = 100K, C1 = 0,33F
Parts:
- C1: value 0.1UF -> 0.33UF
- R1: value 150K -> 100K
- R2: value 56K -> 10K
Changed lines of the file:
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@@
 <part name="JP2" library="pinhead" deviceset="PINHD-1X3" device="/90"/>
 <part name="JP4" library="pinhead" deviceset="PINHD-1X3" device="/90"/>
-<part name="R1" library="resistor" deviceset="R-EU_" device="0207/10" value="150K"/>
-<part name="R2" library="resistor" deviceset="R-EU_" device="0207/10" value="56K"/>
-<part name="C1" library="resistor" deviceset="C-EU" device="025-025X050" value="0.1UF"/>
+<part name="R1" library="resistor" deviceset="R-EU_" device="0207/10" value="100K"/>
+<part name="R2" library="resistor" deviceset="R-EU_" device="0207/10" value="10K"/>
+<part name="C1" library="resistor" deviceset="C-EU" device="025-025X050" value="0.33UF"/>
 <part name="GND7" library="supply1" deviceset="GND" device=""/>
 <part name="JP7" library="pinhead" deviceset="PINHD-1X1" device=""/>
